File: circuits/control/FunctiongeneratorMK3PowerControl.kicad_pcb (KiCad board)
At the start: 2 copper layers, 118.1 x 67.3 mm, 42 parts, among them J1 SIN-TRI-SQU-PWM, J10 12V GND 5V, J11 WaveA2, J12 MO, J2 BTN Range, J3 BTN Form, J4 BTN PWM, J5 FreqRange, J6 WaveA1, J7 FreqCount, J8 Display, J9 14V, K1 G6S-2, Q1 BC337, U1 LTV-847, U2 LM7812_TO220, U3 LM7805_TO220

Commit message: circuit kicad updates
updated circuits to last kicad version

Signed-off-by: Rene Lange <rine@rine.de>
Other:
- net class Default removed
